Commit message: Improve AlohaMini URDF with realistic meshes
- Updated URDF to use STL meshes for gripper base, fingers, and wrist flex components instead of primitive shapes.
- Added STL files to software/src/lerobot/robots/alohamini/meshes/.
- Updated remote_teleop_rerun.py to prefix camera observation keys with 'camera/' to fix Rerun visualization hierarchy errors.

File: software/src/lerobot/robots/alohamini/alohamini.urdf (robot description, URDF)
Before this commit: robot alohamini, 20 links, 19 joints
Links:
- added link left_gripper_finger_2; collision box size=0.04 0.01 0.01; visual mesh filename=meshes/gripper_finger.stl scale=0.001 0.001 0.001
- added link right_gripper_finger_2; collision box size=0.04 0.01 0.01; visual mesh filename=meshes/gripper_finger.stl scale=0.001 0.001 0.001
- link back_wheel: geometry collision cylinder length=0.02 radius=0.05; visual cylinder length=0.02 radius=0.05
- link base_link: mass None -> 10.0
- link left_forearm_link: geometry collision box size=0.15 0.03 0.03; visual box size=0.15 0.03 0.03
- link left_gripper_base_link: geometry collision box size=0.05 0.02 0.04; visual mesh filename=meshes/gripper_base.stl scale=0.001 0.001 0.001
- link left_gripper_finger: geometry collision box size=0.04 0.01 0.01; visual mesh filename=meshes/gripper_finger.stl scale=0.001 0.001 0.001
- link left_shoulder_link: geometry collision box size=0.04 0.04 0.04; visual box size=0.04 0.04 0.04
- link left_shoulder_pan_link: geometry collision cylinder length=0.04 radius=0.02; visual cylinder length=0.04 radius=0.02
- link left_upper_arm_link: geometry collision box size=0.15 0.03 0.03; visual box size=0.15 0.03 0.03
- link left_wheel: geometry collision cylinder length=0.02 radius=0.05; visual cylinder length=0.02 radius=0.05
- link left_wrist_flex_link: geometry collision cylinder length=0.04 radius=0.015; visual mesh filename=meshes/wrist_flex.stl scale=0.001 0.001 0.001
- link lift_base_link: geometry collision box size=0.05 0.05 0.6; visual box size=0.05 0.05 0.6
- link lift_link: mass None -> 0.5; geometry collision box size=0.12 0.05 0.02; visual box size=0.2 0.05 0.02
- link right_forearm_link: geometry collision box size=0.15 0.03 0.03; visual box size=0.15 0.03 0.03
- link right_gripper_base_link: geometry collision box size=0.05 0.02 0.04; visual mesh filename=meshes/gripper_base.stl scale=0.001 0.001 0.001
- link right_gripper_finger: geometry collision box size=0.04 0.01 0.01; visual mesh filename=meshes/gripper_finger.stl scale=0.001 0.001 0.001
- link right_shoulder_link: geometry collision box size=0.04 0.04 0.04; visual box size=0.04 0.04 0.04
- link right_shoulder_pan_link: geometry collision cylinder length=0.04 radius=0.02; visual cylinder length=0.04 radius=0.02
- link right_upper_arm_link: geometry collision box size=0.15 0.03 0.03; visual box size=0.15 0.03 0.03
- link right_wheel: geometry collision cylinder length=0.02 radius=0.05; visual cylinder length=0.02 radius=0.05
- link right_wrist_flex_link: geometry collision cylinder length=0.04 radius=0.015; visual mesh filename=meshes/wrist_flex.stl scale=0.001 0.001 0.001
Joints:
- added joint arm_left_gripper_2: type revolute, parent left_gripper_base_link, child left_gripper_finger_2, origin xyz=0.05 -0.02 0 rpy=0 0 0, axis 0 0 -1, limit lower=-1.0 upper=1.0 effort=5 velocity=5.0
- added joint arm_right_gripper_2: type revolute, parent right_gripper_base_link, child right_gripper_finger_2, origin xyz=0.05 -0.02 0 rpy=0 0 0, axis 0 0 -1, limit lower=-1.0 upper=1.0 effort=5 velocity=5.0
- joint arm_left_gripper: origin xyz=0.05 0 0 rpy=0 0 0 -> xyz=0.05 0.02 0 rpy=0 0 0
- joint arm_right_gripper: origin xyz=0.05 0 0 rpy=0 0 0 -> xyz=0.05 0.02 0 rpy=0 0 0
